File: hardware/PCB/esp32_hitbox_v1.0.0/esp32_hitbox_v1.0.0.kicad_pcb (KiCad board)
At the start: 2 copper layers, 16 parts

Commit message: update sch
Parts:
- removed SW1, SW10, SW11, SW12, SW13, SW14, SW15, SW16, SW2, SW3, SW4, SW5, SW6, SW7, SW8, SW9: ~, DuRuofu_Switch:Shaft_Base
- added U1: ~, DuRuofu_Switch:热插拔键盘轴(RGB反贴)(30mm), F.Cu at (81.8, 45.0)
- added U10: ~, DuRuofu_Switch:热插拔键盘轴(RGB反贴)(30mm), F.Cu at (235.5, 80.5)
- added U11: ~, DuRuofu_Switch:热插拔键盘轴(RGB反贴)(30mm), F.Cu at (180.8, 55.4)
- added U12: ~, DuRuofu_Switch:热插拔键盘轴(RGB反贴)(30mm), F.Cu at (180.8, 82.0)
- added U13: ~, DuRuofu_Switch:热插拔键盘轴(RGB反贴)(30mm), F.Cu at (111.3, 125.0)
- added U14: ~, DuRuofu_Switch:热插拔键盘轴(RGB反贴)(30mm), F.Cu at (138.4, 124.5)
- added U2: ~, DuRuofu_Switch:热插拔键盘轴(RGB反贴)(30mm), F.Cu at (47.0, 77.5)
- added U3: ~, DuRuofu_Switch:热插拔键盘轴(RGB反贴)(30mm), F.Cu at (74.9, 73.7)
- added U4: ~, DuRuofu_Switch:热插拔键盘轴(RGB反贴)(30mm), F.Cu at (101.6, 84.8)
- added U5: ~, DuRuofu_Switch:热插拔键盘轴(RGB反贴)(30mm), F.Cu at (235.5, 53.8)
- added U6: ~, DuRuofu_Switch:热插拔键盘轴(RGB反贴)(30mm), F.Cu at (154.9, 63.6)
- added U7: ~, DuRuofu_Switch:热插拔键盘轴(RGB反贴)(30mm), F.Cu at (154.9, 90.2)
- added U8: ~, DuRuofu_Switch:热插拔键盘轴(RGB反贴)(30mm), F.Cu at (208.3, 52.7)
- added U9: ~, DuRuofu_Switch:热插拔键盘轴(RGB反贴)(30mm), F.Cu at (208.3, 79.3)
Other:
- board outline added: 230.5 x 170 mm
