File: hardware/PCB/esp32_hitbox_v1.0.0/esp32_hitbox_v1.0.0.kicad_sch (KiCad schematic)
At the start: 16 parts

Commit message: update sch
Parts:
- removed SW1, SW10, SW11, SW12, SW13, SW14, SW15, SW16, SW2, SW3, SW4, SW5, SW6, SW7, SW8, SW9: ~, DuRuofu_Switch:Shaft_Base, symbol Switch:SW_Push
- added U1, U10, U11, U12, U13, U14, U2, U3, U4, U5, U6, U7, U8, U9: ~, DuRuofu_Switch:热插拔键盘轴(RGB反贴)(30mm), symbol DuRuofu_Switch:机械键盘按键(RGB)
